Commit message: modified k3hand_slider

File: urdf/robot.urdf (robot description, URDF)
Before this commit: robot firefighter, 16 links, 15 joints
Joints:
- removed joint joint_fin1_1
- removed joint joint_fin1_2
- removed joint joint_fin1_3
- removed joint joint_fin1_4
- removed joint joint_fin2_1
- removed joint joint_fin2_2
- removed joint joint_fin3_1
- removed joint joint_fin3_2
- added joint joint0: type revolute, parent palm, child link_fin2_1, origin xyz=0.020 -0.015 0.020 rpy=0.0 0.0 1.570796, axis 0.0 0.0 1.0, limit lower=-1.570796 upper=0.523599 effort=0.0 velocity=0.0
- added joint joint1: type revolute, parent link_fin2_1, child link_fin2_2, origin xyz=0.000 -0.020 0.0 rpy=-1.570796 0.0 0.0, axis 1.0 0.0 0, limit lower=-1.570796 upper=1.579796 effort=0.0 velocity=0.0
- added joint joint2: type revolute, parent palm, child link_fin3_1, origin xyz=-0.020 -0.015 0.020 rpy=0.0 0.0 -1.570796, axis 0.0 0.0 1.0, limit lower=-0.523599 upper=1.570796 effort=0.0 velocity=0.0
- added joint joint3: type revolute, parent link_fin3_1, child link_fin3_2, origin xyz=0.000 -0.020 0.0 rpy=-1.570796 0.0 0.0, axis -1.0 0.0 0, limit lower=-1.570796 upper=1.570796 effort=0.0 velocity=0.0
- added joint joint4: type revolute, parent palm, child link_fin1_1, origin xyz=0 0.02 0 rpy=0.78537 0 0, axis 0.0 0 -1, limit lower=-1.570796 upper=1.570796 effort=30.0 velocity=1.0
- added joint joint5: type revolute, parent link_fin1_1, child link_fin1_2, origin xyz=0 0.0275 0 rpy=-0.78537 0 0, axis 1 0.0 0.0, limit lower=-0.8726646 upper=2.268928 effort=0.0 velocity=0.0
- added joint joint6: type revolute, parent link_fin1_2, child link_fin1_3, origin xyz=0 0.035 0 rpy=0 0 0, axis 1 0.0 0.0, limit lower=-1.570796 upper=1.570796 effort=0.0 velocity=0.0
- added joint joint7: type revolute, parent link_fin1_3, child link_fin1_4, origin xyz=0 0.035 0 rpy=0 0 0, axis 1 0.0 0.0, limit lower=-1.570796 upper=1.570796 effort=0.0 velocity=0.0
