Commit message: change urdf

File: urdf/k3hand.urdf (robot description, URDF)
Before this commit: robot myfirst, 9 links, 8 joints
Links:
- link base_link: mass 10 -> None; geometry collision cylinder length=0.06 radius=0.025; visual mesh filename=package://k3hand_ros/urdf/hand/palm.stl
- link link_fin2_1: geometry collision box size=0.020 0.030 0.012; visual mesh filename=package://k3hand_ros/urdf/hand/link_fin1_1.stl

File: urdf/robot.urdf (robot description, URDF)
Before this commit: robot firefighter, 16 links, 15 joints
Links:
- link base_link: geometry collision cylinder length=0.102 radius=0.0725; visual mesh filename=package://k3hand_ros/urdf/320_urdf/base.dae

Commit message: add .dae file to urdf

File: urdf/k3hand.urdf (robot description, URDF)
Before this commit: robot myfirst, 9 links, 8 joints
Links:
- removed link link_fin1_1
- removed link link_fin1_2
- removed link link_fin1_3
- removed link link_fin1_4
- removed link link_fin2_1
- removed link link_fin2_2
- removed link link_fin3_1
- removed link link_fin3_2
- added link fing_met_1, mass 10; collision box size=0.020 0.030 0.012; visual mesh filename=package://k3hand_ros/urdf/k3_urdf/fing_met_1.dae
- added link fing_met_2, mass 10; collision box size=0.020 0.030 0.012; visual mesh filename=package://k3hand_ros/urdf/k3_urdf/fing_met_2.dae
- added link fing_middle_1, mass 10; collision box size=0.020 0.120 0.012; visual mesh filename=package://k3hand_ros/urdf/k3_urdf/fing_middle_1.dae
- added link fing_middle_2, mass 10; collision box size=0.020 0.120 0.012; visual mesh filename=package://k3hand_ros/urdf/k3_urdf/fing_middle_2.dae
- added link thumb_met, mass 10; collision box size=0.0225 0.035 0.012; visual mesh filename=package://k3hand_ros/urdf/k3_urdf/thumb_met.dae
- added link thumb_middle_1, mass 10; collision box size=0.0225 0.045 0.012; visual mesh filename=package://k3hand_ros/urdf/k3_urdf/thumb_middle_1.dae
- added link thumb_middle_2, mass 10; collision box size=0.0225 0.045 0.012; visual mesh filename=package://k3hand_ros/urdf/k3_urdf/thumb_middle_2.dae
- added link thumb_tip, mass 10; collision box size=0.0225 0.040 0.012; visual mesh filename=package://k3hand_ros/urdf/k3_urdf/thumb_tip.dae
- added link wrist; collision cylinder length=0.06 radius=0.025; visual mesh filename=package://k3hand_ros/urdf/k3_urdf/wrist.dae
- link base_link: geometry 
Joints:
- added joint base2wrist: type fixed, parent base_link, child wrist, origin xyz=0 0 0 rpy=0 0 0
- joint joint0: axis 0.0 0.0 1.0 -> 0.0 1.0 0.0; child link_fin2_1 -> fing_met_1; origin xyz=0.020 -0.015 0.020 rpy=0.0 0.0 1.570796 -> xyz=0.0225 -0.0175 0.00 rpy=0.0 1.570796 0.0; parent base_link -> wrist
- joint joint1: child link_fin2_2 -> fing_middle_1; parent link_fin2_1 -> fing_met_1
- joint joint2: child link_fin3_1 -> fing_met_2; parent base_link -> wrist
- joint joint3: child link_fin3_2 -> fing_middle_2; parent link_fin3_1 -> fing_met_2
- joint joint4: child link_fin1_1 -> thumb_met; parent base_link -> wrist
- joint joint5: child link_fin1_2 -> thumb_middle_1; origin xyz=0 0.0275 0 rpy=-0.78537 0 0 -> xyz=0 0.0 0 rpy=-0.78537 0 0; parent link_fin1_1 -> thumb_met
- joint joint6: child link_fin1_3 -> thumb_middle_2; origin xyz=0 0.035 0 rpy=0 0 0 -> xyz=0 0.0 0 rpy=0 0 0; parent link_fin1_2 -> thumb_middle_1
- joint joint7: child link_fin1_4 -> thumb_tip; origin xyz=0 0.035 0 rpy=0 0 0 -> xyz=0 0 0 rpy=0 0 0; parent link_fin1_3 -> thumb_middle_2

Commit message: add dae file and change urdf file

File: urdf/k3hand.urdf (robot description, URDF)
Before this commit: robot myfirst, 10 links, 9 joints
Links:
- added link fing_base_1, mass 10; collision box size=0.030 0.03 0.05; visual mesh filename=package://k3hand_ros/urdf/k3_urdf/fing_base_1.dae
- added link fing_base_2, mass 10; collision box size=0.030 0.03 0.05; visual mesh filename=package://k3hand_ros/urdf/k3_urdf/fing_base_2.dae
- added link fing_tip_1, mass 10; collision box size=0.020 0.015 0.02; visual mesh filename=package://k3hand_ros/urdf/k3_urdf/fing_tip_1.dae
- added link fing_tip_2, mass 10; collision box size=0.020 0.015 0.02; visual mesh filename=package://k3hand_ros/urdf/k3_urdf/fing_tip_2.dae
- link fing_met_1: geometry collision box size=0.020 0.012 0.03; visual mesh filename=package://k3hand_ros/urdf/k3_urdf/fing_met_1.dae
- link fing_met_2: geometry collision box size=0.020 0.0120 0.03; visual mesh filename=package://k3hand_ros/urdf/k3_urdf/fing_met_2.dae
- link fing_middle_1: geometry collision box size=0.020 0.03 0.05; visual mesh filename=package://k3hand_ros/urdf/k3_urdf/fing_middle_1.dae
- link fing_middle_2: geometry collision box size=0.020 0.03 0.05; visual mesh filename=package://k3hand_ros/urdf/k3_urdf/fing_middle_2.dae
- link thumb_middle_1: geometry collision box size=0.0225 0.012 0.05; visual mesh filename=package://k3hand_ros/urdf/k3_urdf/thumb_middle_1.dae
- link thumb_middle_2: geometry collision box size=0.0225 0.012 0.05; visual mesh filename=package://k3hand_ros/urdf/k3_urdf/thumb_middle_2.dae
- link thumb_tip: geometry collision box size=0.0225 0.015 0.040; visual mesh filename=package://k3hand_ros/urdf/k3_urdf/thumb_tip.dae
Joints:
- removed joint joint0
- removed joint joint1
- removed joint joint2
- removed joint joint3
- removed joint joint4
- removed joint joint5
- removed joint joint6
- removed joint joint7
- added joint fing_fixed_joint_1_1: type fixed, parent fing_base_1, child fing_middle_1, origin xyz=0 0 0.0 rpy=0 0 0
- added joint fing_fixed_joint_1_2: type fixed, parent fing_middle_1, child fing_tip_1, origin xyz=0 0 0.0 rpy=0 0 0
- added joint fing_fixed_joint_2_1: type fixed, parent fing_base_2, child fing_middle_2, origin xyz=0 0 0.0 rpy=0 0 0
- added joint fing_fixed_joint_2_2: type fixed, parent fing_middle_2, child fing_tip_2, origin xyz=0 0 0.0 rpy=0 0 0
- added joint hand_joint_0: type revolute, parent wrist, child fing_met_1, origin xyz=-0.0225 -0.0225 0.00 rpy=0 -1.570796 0, axis 0.0 -1.0 0.0, limit lower=-1.570796 upper=0.523599 effort=0.0 velocity=0.0
- added joint hand_joint_1: type revolute, parent fing_met_1, child fing_base_1, origin xyz=0.0075 -0.0 0.022 rpy=1.570796 0.0 0.0, axis 1.0 0.0 0, limit lower=-1.570796 upper=1.579796 effort=0.0 velocity=0.0
- added joint hand_joint_2: type revolute, parent wrist, child fing_met_2, origin xyz=0.0225 -0.0225 0.00 rpy=0.0 1.570796 0, axis 0.0 1.0 0.0, limit lower=-0.523599 upper=1.570796 effort=0.0 velocity=0.0
- added joint hand_joint_3: type revolute, parent fing_met_2, child fing_base_2, origin xyz=-0.0075 -0.0 0.022 rpy=1.570796 0.0 0.0, axis -1.0 0.0 0, limit lower=-1.570796 upper=1.570796 effort=0.0 velocity=0.0
- added joint hand_joint_4: type revolute, parent wrist, child thumb_met, origin xyz=0 -0.0080 -0.043 rpy=0 0 0, axis 0.0 1 -1.21, limit lower=-1.570796 upper=1.570796 effort=30.0 velocity=1.0
- added joint hand_joint_5: type revolute, parent thumb_met, child thumb_middle_1, origin xyz=0 -0.0145 -0.0177 rpy=0 0 0, axis -1 0.0 0.0, limit lower=-0.8726646 upper=2.268928 effort=0.0 velocity=0.0
- added joint hand_joint_6: type revolute, parent thumb_middle_1, child thumb_middle_2, origin xyz=0 0.0 -0.0358 rpy=0 0 0, axis 1 0.0 0.0, limit lower=-1.570796 upper=1.570796 effort=0.0 velocity=0.0
- added joint hand_joint_7: type revolute, parent thumb_middle_2, child thumb_tip, origin xyz=0 0 -0.036 rpy=0 0 0, axis 1 0.0 0.0, limit lower=-1.570796 upper=1.570796 effort=0.0 velocity=0.0
